File: Hardware/ETH1CREF1C/ADC.kicad_sch (KiCad schematic)
At the start: 58 parts, among them Q503 BC847, U501 DG211B, U502 OPA2192, U503 DG419xY, U505 LT5400-100k-100k, U506 LM399H, U507 LT5400-5k-1k, U508 OPA177, U509 OPA140, U511 OPA192, U512 LT5400-10k-10k, U513 LM311

Commit message: Hardware
Parts:
- R306: renamed from R510; value 62/.1% -> 62
- gave numbers to parts that had none: 1
- renumbered C502 to C301, C503 to C302, C504 to C303, C505 to C304, C506 to C305, C507 to C306, C508 to C307, C509 to C308, C510 to C309, C511 to C310, C512 to C311, C513 to C312, C514 to C313, C515 to C314, C516 to C315, C517 to C316, C518 to C317, C519 to C318, C520 to C319, C521 to C320, C522 to C321, C523 to C322, C524 to C323, D503 to D301, D504 to D302, D505 to D303, Q503 to Q301, R503 to R301, R505 to R302, R506 to R303, R507 to R304, R509 to R305, R511 to R308, R512 to R309, R514 to R310, R517 to R311, R518 to R312, R519 to R313, R520 to R314, R522 to R315, R523 to R316, R524 to R317, R525 to R318, R526 to R319, R527 to R320, U501 to U301, U502 to U302, U503 to U303, U505 to U304, U506 to U305, U507 to U306, U508 to U307, U509 to U308, U511 to U309, U512 to U310, U513 to U311
Connections:
- net DGNDF is gone; now on net GND: C319.2, C322.2, U311.1 (GND)
- net at R306.2, U305.2: no longer U307.3 (+)
- net at C310.1, R305.1, R306.1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: now also U307.3 (+)
- net +3.3VP renamed +3V3
- net +5VF renamed +5V
- net AGNDF renamed GND
Other:
- moved on the sheet: C310, C313, C314, C320, C321, C323, D301, D302, D303, Q301, R301, R302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
