File: Hardware/ETH1CREF1C/FPGA.kicad_sch (KiCad schematic)
At the start: 64 parts, among them J801 Conn_01x04_Male, J802 Conn_02x05, Q801 BC857, U801 SN74LVC1T45DBV, U802 SN74LVC1T45DBV, U803 ICE40HX4K-TQ144, U804 SN74LVC1T45DBV, U805 SN74LVC1T45DBV, U806 SN74LVC1T45DBV, U807 SN74LVC1T45DBV, U808 ASDMB-100.000MHZ, U809 MT25QL128ABA1ESE

Commit message: Hardware
Parts:
- added C202: 4u7, symbol Device:C
- added U201: MCP1700T-1202E/TT, Package_TO_SOT_SMD:SOT-23, symbol Regulator_Linear:MCP1700x-120xxTT
- renumbered C801 to C201, C802 to C203, C803 to C204, C804 to C205, C805 to C206, C806 to C207, C807 to C208, C808 to C209, C809 to C210, C810 to C211, C811 to C212, C812 to C213, C813 to C214, C814 to C215, C815 to C216, C816 to C217, C817 to C218, C818 to C219, C819 to C220, C820 to C221, C821 to C222, C822 to C223, C823 to C224, C824 to C225, C825 to C226, C826 to C227, C827 to C228, C828 to C229, C829 to C230, C830 to C231, D801 to D201, D802 to D202, D803 to D203, J801 to J201, J802 to J202, Q801 to Q201, R801 to R201, R802 to R202, R803 to R203, R804 to R204, R805 to R205, R806 to R206, R807 to R207, R808 to R208, R809 to R209, R810 to R210, R811 to R211, R812 to R212, R813 to R213, R814 to R214, R815 to R215, R816 to R216, R817 to R217, R818 to R218, R819 to R219, U801 to U202, U802 to U203, U803 to U204, U804 to U205, U805 to U206, U806 to U207, U807 to U208, U808 to U209, U809 to U210
Connections:
- net +1V2: now also U201.2 (VO)
- net +3.3VP renamed +3V3
- net +5VF renamed +5V
- net DGNDF renamed GND
- net GND: now also C202.2, U201.1 (GND)
- new net +3.3V: C202.1, U201.3 (VI)
Other:
- moved on the sheet: C201, C203, C204, C205, C206, C207, C208, C209, C210, C211, C212, C213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
