File: Hardware/ETH1CREF1C/Input.kicad_sch (KiCad schematic)
At the start: 63 parts, among them K603 HE3621A0510, Q601 BC847, Q602 BC857, U601 DG211B, U602 DG211B, U603 SN74LVC1T45DBV, U604 SN74LVC1T45DBV, U605 SN74LVC1T45DBV, U606 74HCT595, U607 74HCT595, U608 LTC1052, U609 AD711, U610 AD711, U611 TL431DBZ, U612 TL431DBZ, U613 LT5400-9k-1k

Commit message: Hardware
Parts:
- renumbered C601 to C401, C602 to C402, C603 to C403, C604 to C404, C605 to C405, C606 to C406, C607 to C407, C608 to C408, C609 to C409, C610 to C410, C611 to C411, C612 to C412, C613 to C413, C614 to C414, C615 to C415, C616 to C416, C617 to C417, C618 to C418, C619 to C419, C620 to C420, C621 to C421, C622 to C422, C623 to C423, C624 to C424, C625 to C425, K603 to K401, L601 to L401, Q601 to Q401, Q602 to Q402, R610 to R401, R611 to R402, R612 to R403, R613 to R404, R614 to R405, R615 to R406, R616 to R407, R617 to R408, R618 to R409, R619 to R410, R620 to R411, R621 to R412, R622 to R413, R623 to R414, R624 to R415, R625 to R416, R626 to R417, R627 to R418, R628 to R419, R629 to R420, R630 to R421, U601 to U401, U602 to U402, U603 to U403, U604 to U404, U605 to U405, U606 to U406, U607 to U407, U608 to U408, U609 to U409, U610 to U410, U611 to U411, U612 to U412, U613 to U413
Connections:
- net DGNDF is gone; now on net GND: C403.2, C405.2, C406.2, C407.2, C408.2, C409.2, C411.2, C412.2, C413.2, C414.2, U403.2 (GND), U403.5 (DIR), U404.2 (GND), U404.5 (DIR), U405.2 (GND), U405.5 (DIR), U406.13 (~{OE}), U406.8 (GND), U407.13 (~{OE}), U407.8 (GND)
- net +3.3VF renamed +3.3V
- net +5VF renamed +5V
- net AGNDF renamed GND
